File: HARDWARE/Hardware revision G/ESP32-GATEWAY_Rev_G.kicad_pcb (KiCad board)
At the start: 2 copper layers, 50.8 x 62.2 mm, 101 parts, among them CON1 NA(NH1x20), Q3 Q12MHz/20pF/30ppm/2P/HC-49SM(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, Q4 BC817-40(SOT23), Q5 BC817-40(SOT23), T1 DTC114YKA, U2 SY8089AAAC(SOT23-5), U3 ESP32-WROOM-32D-4MB, U4 LAN8710A-EZC(QFN32), U5 CH340T(SSOP20W)

Commit message: Update ESP32-GATEWAY_Rev_G.kicad_pcb
Parts:
- BUT1, RST1: footprint OLIMEX_Buttons-FP:T1107A(6x3,8x2,5MM) -> VADACTRO_Buttons-FP:T1107A(6x3,8x2,5MM)
- C1, C10, C3, C4: footprint OLIMEX_RLC-FP:C_0805_5MIL_DWS -> VADACTRO_RLC-FP:C_0805_5MIL_DWS
- C11, C12, C13, C14, C15, C16, C17, C18, C2, C21, C22, C23, C24, C8, C9: footprint OLIMEX_RLC-FP:C_0603_5MIL_DWS -> VADACTRO_RLC-FP:C_0603_5MIL_DWS
- C19, C20: footprint OLIMEX_RLC-FP:C_1206_5MIL_DWS_ISO -> VADACTRO_RLC-FP:C_1206_5MIL_DWS_ISO
- CON1: footprint OLIMEX_Connectors-FP:HN1x20 -> VADACTRO_Connectors-FP:HN1x20
- D1, D3: footprint OLIMEX_Diodes-FP:SOD-123_1C-2A_KA -> VADACTRO_Diodes-FP:SOD-123_1C-2A_KA
- D2: footprint OLIMEX_Diodes-FP:DO214AA_1(K)-2(A) -> VADACTRO_Diodes-FP:DO214AA_1(K)-2(A)
- D4: footprint OLIMEX_Diodes-FP:SOT23-3 -> VADACTRO_Diodes-FP:SOT23-3
- D6: footprint OLIMEX_Diodes-FP:SMA-KA -> VADACTRO_Diodes-FP:SMA-KA
- FET1, FET2, Q4, Q5, T1: footprint OLIMEX_Transistors-FP:SOT23 -> VADACTRO_Transistors-FP:SOT23
- FID1, FID2, FID3: footprint OLIMEX_Other-FP:Fiducial1x3 -> VADACTRO_Other-FP:Fiducial1x3
- GND1: footprint OLIMEX_Other-FP:TESTPAD_40-ROUND -> VADACTRO_Other-FP:TESTPAD_40-ROUND
- L1, L3, L4: footprint OLIMEX_RLC-FP:L_0805_5MIL_DWS -> VADACTRO_RLC-FP:L_0805_5MIL_DWS
- L2: footprint OLIMEX_RLC-FP:CD32 -> VADACTRO_RLC-FP:CD32
- LAN1: footprint OLIMEX_Connectors-FP:RJLBC-060TC1 -> VADACTRO_Connectors-FP:RJLBC-060TC1
- LED1, PWRLED1: footprint OLIMEX_LEDs-FP:LED_0603_KA -> VADACTRO_LEDs-FP:LED_0603_KA
- LED_E1, PHY_RST1: footprint OLIMEX_Jumpers-FP:SJ -> VADACTRO_Jumpers-FP:SJ
- Logo-OLimeX: footprint OLIMEX_LOGOs-FP:OLIMEX_LOGO_TB -> VADACTRO_LOGOs-FP:OLIMEX_LOGO_TB
- Logo-OSHW: footprint OLIMEX_LOGOs-FP:LOGO_OPENHARDWARE_8x8 -> VADACTRO_LOGOs-FP:LOGO_OPENHARDWARE_8x8
- Logo-vadactroBIG: renamed from Logo-OlimexBIG; footprint OLIMEX_LOGOs-FP:OLIMEX_LOGO_TB -> VADACTRO_LOGOs-FP:VADACTRO_LOGO_TB
- MH1, MH2: footprint OLIMEX_Other-FP:Mounting_hole_Shield_3.3mm -> VADACTRO_Other-FP:Mounting_hole_Shield_3.3mm
- MICRO_SD1: footprint OLIMEX_Connectors-FP:TFC-WXCP11-08-LF -> VADACTRO_Connectors-FP:TFC-WXCP11-08-LF
- Q3: footprint OLIMEX_Crystal-FP:Q_49U3HMS -> VADACTRO_Crystal-FP:Q_49U3HMS
- R1, R10, R11, R14, R16, R19, R2, R20, R24, R25, R26, R27, R28, R29, R3, R30, R31, R32, R33, R35, R37, R38, R39, R4, R40, R41, R42, R43, R45, R46, R5, R6, R7, R8, R9: footprint OLIMEX_RLC-FP:R_0603_5MIL_DWS -> VADACTRO_RLC-FP:R_0603_5MIL_DWS
- RM2, RM3: footprint OLIMEX_RLC-FP:R_MATRIX_4 -> VADACTRO_RLC-FP:R_MATRIX_4
- Sign-Antistatic: footprint OLIMEX_LOGOs-FP:LOGO_ANTISTATIC_1 -> VADACTRO_LOGOs-FP:LOGO_ANTISTATIC_1
- Sign-RecyclBin: footprint OLIMEX_LOGOs-FP:LOGO_RECYCLEBIN_1 -> VADACTRO_LOGOs-FP:LOGO_RECYCLEBIN_1
- Sign_Pb-Free: footprint OLIMEX_LOGOs-FP:LOGO_PBFREE -> VADACTRO_LOGOs-FP:LOGO_PBFREE
- Sign_RoHS: footprint OLIMEX_LOGOs-FP:LOGO_ROHS_1 -> VADACTRO_LOGOs-FP:LOGO_ROHS_1
- U2: footprint OLIMEX_Regulators-FP:SOT-23-5 -> VADACTRO_Regulators-FP:SOT-23-5
- U3: footprint OLIMEX_Cases-FP:ESP-WROOM-32_MODULE -> VADACTRO_Cases-FP:ESP-WROOM-32_MODULE
- U4: footprint OLIMEX_IC-FP:QFN32_EP(33)_5.00x5.00x0.90mm_Pitch_0.50mm -> VADACTRO_IC-FP:QFN32_EP(33)_5.00x5.00x0.90mm_Pitch_0.50mm
- U5: footprint OLIMEX_IC-FP:SSOP-20W -> VADACTRO_IC-FP:SSOP-20W
- USB-UART1: footprint OLIMEX_Connectors-FP:USB-MICRO_MISB-SWMM-5B_LF -> VADACTRO_Connectors-FP:USB-MICRO_MISB-SWMM-5B_LF
